File: mcu_datalogger/mcu_datalogger.kicad_pcb (KiCad board)
At the start: 2 copper layers, 29 parts, among them J1 Conn_01x04_Pin, J2 Conn_01x04_Pin, J3 Conn_01x09_Pin, J4 Conn_02x03_Odd_Even, U1 24LC1025, U2 24LC1025, U3 DS1337S_, U4 ATMEGA328P-AU, Y1 32.768 KHz, Y2 16 MHz

Commit message: layout / organization
Parts:
- moved J3 94.9 mm to (76.8, 99.7), turned to 90 degrees
- moved Y1 88.1 mm to (71.1, 86.4), turned to 90 degrees
- moved BT1 85.8 mm to (71.1, 76.2)
- moved U3 85.4 mm to (78.7, 73.0)
- moved J1 74.9 mm to (102.2, 99.7), turned to 90 degrees
- moved U2 71.9 mm to (78.7, 88.3)
- moved U1 71.8 mm to (78.7, 80.6)
- moved Y2 71.0 mm to (88.6, 87.7), turned to 180 degrees
- moved J4 68.0 mm to (107.1, 71.6)
- moved R3 63.9 mm to (76.8, 92.7)
- moved H4 63.6 mm to (71.1, 99.1)
- moved H1 63.5 mm to (71.1, 71.1)
- moved D2 63.3 mm to (98.6, 71.0)
- moved U4 61.6 mm to (88.4, 79.5)
- moved R2 60.5 mm to (80.9, 92.7)
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
Commit message: routing pt 1
Routing:
- net /VCC: track 0.00 -> 202.1 mm, vias 0 -> 15
- net GND: track 0.00 -> 148.0 mm, vias 0 -> 5
- net /MOSI: track 0.00 -> 137.8 mm, vias 0 -> 2
- net /SCK: track 0.00 -> 135.9 mm, vias 0 -> 7
- net /SDA: track 0.00 -> 107.2 mm, vias 0 -> 4
- net Net-(BT1-+): track 0.00 -> 60.1 mm, vias 0 -> 5
- net /TX: track 0.00 -> 53.4 mm, vias 0 -> 1
- net /RX: track 0.00 -> 49.3 mm, vias 0 -> 1
- net /MISO: track 0.00 -> 32.7 mm, vias 0 -> 2
- net Net-(U3-SQW/~INT): track 0.00 -> 32.5 mm
- net Net-(U3-~{INTA}): track 0.00 -> 27.2 mm
- net Net-(U4-PB6): track 0.00 -> 26.2 mm
- net /RESET: track 0.00 -> 24.2 mm
- net Net-(U3-X2): track 0.00 -> 19.7 mm
- net Net-(U4-PB7): track 0.00 -> 19.1 mm
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
Commit message: routing pt 2
finished most of the routuing, only one error on drc
Routing:
- net /D2: track 1.39 -> 72.2 mm
- net /D4: track 0.00 -> 67.0 mm, vias 0 -> 1
- net GND: track 148.0 -> 211.5 mm, vias 5 -> 11
- net /D3: track 0.00 -> 62.7 mm, vias 0 -> 1
- net Net-(U4-PB6): track 26.2 -> 84.3 mm
- net /D8: track 0.00 -> 32.8 mm, vias 0 -> 1
- net /D7: track 0.00 -> 30.7 mm, vias 0 -> 1
- net /D6: track 0.00 -> 28.4 mm, vias 0 -> 1
- net /D5: track 0.00 -> 25.6 mm, vias 0 -> 1
- net /VCC: track 202.1 -> 218.3 mm, vias 15 -> 17
- net Net-(BT1-+): track 60.1 -> 69.0 mm, vias 5 -> 4
- net /SDA: track 107.2 -> 108.1 mm
- net /SCK: track 135.9 -> 136.5 mm

Commit message: fix drc error
Other:
- board outline added: 57 x 36.7 mm
Changed lines of the file:
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@@
 		)
 		(property "Value" "Battery"
-			(at 0 4.92 0)
+			(at 0.762 4.8768 0)
 			(layer "F.Fab")
 			(effects
@@
 		)
 		(property "Value" "MountingHole"
-			(at 0 3.05 0)
+			(at -6.8072 -1.524 0)
 			(layer "F.Fab")
 			(effects
@@
 		)
 		(property "Value" "Conn_01x09_Pin"
-			(at 0 22.7 90)
+			(at 2.921 16.0274 180)
 			(layer "F.Fab")
 			(effects
@@
 		)
 		(property "Value" "MountingHole"
-			(at 0 3.05 0)
+			(at 7.5692 -2.4384 0)
 			(layer "F.Fab")
 			(effects
@@
 		)
 		(property "Value" "Conn_01x04_Pin"
-			(at 0 10 90)
+			(at 2.9718 6.2738 180)
 			(layer "F.Fab")
 			(effects
@@
 		)
 		(property "Value" "MountingHole"
-			(at 0 3.05 0)
+			(at -5.2324 -3.8608 0)
 			(layer "F.Fab")
 			(effects
@@
 		)
 		(property "Value" "Conn_01x04_Pin"
-			(at 0 10 0)
+			(at -2.9464 8.0264 270)
 			(layer "F.Fab")
 			(effects
@@
 		)
 		(property "Value" "MountingHole"
-			(at 0 3.05 0)
+			(at 7.6708 -1.0668 0)
 			(layer "F.Fab")
 			(effects
@@
 		(net "Net-(U4-PB6)")
 	)
+	(gr_rect
+		(start 64.9732 67.0052)
+		(end 122.0216 103.6828)
+		(stroke
+			(width 0.05)
+			(type default)
+		)
+		(fill no)
+		(layer "Edge.Cuts")
+	)
 	(segment
 		(start 75.14 91.65)
@@
 	)
 	(segment
-		(start 90.847426 79.233425)
-		(end 90.495955 79.584896)
+		(start 79.587184 81.556)
+		(end 74.114001 81.556)
 		(width 0.2)
 		(layer "B.Cu")
@@
 	)
 	(segment
-		(start 79.587184 81.556)
-		(end 74.114001 81.556)
+		(start 89.6112 79.3432)
+		(end 89.538 79.3432)
 		(width 0.2)
 		(layer "B.Cu")
@@
 	)
 	(segment
-		(start 89.6112 79.3432)
-		(end 89.538 79.3432)
+		(start 75.519315 98.145)
+		(end 78.150685 98.145)
 		(width 0.2)
 		(layer "B.Cu")
@@
 	)
 	(segment
-		(start 74.3584 99.00823)
-		(end 74.47163 98.895)
+		(start 78.385 98.379315)
+		(end 78.385 100.222114)
 		(width 0.2)
 		(layer "B.Cu")
@@
 	)
 	(segment
-		(start 74.47163 98.895)
-		(end 75.285 98.895)
+		(start 72.024913 81.2292)
+		(end 70.215087 81.2292)
 		(width 0.2)
 		(layer "B.Cu")
@@
 	)
 	(segment
-		(start 80.485586 80.6576)
-		(end 79.587184 81.556)
+		(start 74.114001 81.556)
+		(end 73.914 81.355999)
 		(width 0.2)
 		(layer "B.Cu")
@@
 	)
 	(segment
-		(start 73.914 81.355999)
-		(end 73.447571 81.355999)
+		(start 89.538 79.713901)
+		(end 88.594299 80.6576)
 		(width 0.2)
 		(layer "B.Cu")
@@
 	)
 	(segment
-		(start 73.447571 81.355999)
-		(end 72.672842 80.581271)
+		(start 79.357886 99.695)
+		(end 79.375 99.695)
 		(width 0.2)
 		(layer "B.Cu")
@@
 	)
 	(segment
-		(start 72.672842 80.581271)
-		(end 72.114112 81.14)
+		(start 90.495955 79.584896)
+		(end 89.852896 79.584896)
 		(width 0.2)
 		(layer "B.Cu")
@@
 	)
 	(segment
-		(start 78.385 100.222114)
-		(end 78.607886 100.445)
+		(start 89.852896 79.584896)
+		(end 89.6112 79.3432)
 		(width 0.2)
 		(layer "B.Cu")
@@
 	)
 	(segment
-		(start 70.125887 81.14)
-		(end 69.6848 80.698913)
+		(start 73.549729 96.802357)
+		(end 73.803728 96.802357)
 		(width 0.2)
 		(layer "B.Cu")
@@
 	)
 	(segment
-		(start 72.114112 81.14)
-		(end 70.125887 81.14)
+		(start 78.607886 100.445)
+		(end 79.357886 99.695)
 		(width 0.2)
 		(layer "B.Cu")
@@
 	)
 	(segment
-		(start 74.3584 97.35703)
-		(end 74.3584 99.00823)
+		(start 75.285 98.895)
+		(end 75.285 98.379315)
 		(width 0.2)
 		(layer "B.Cu")
@@
 	)
 	(segment
-		(start 73.803728 96.802357)
-		(end 74.3584 97.35703)
+		(start 90.847426 78.736367)
+		(end 90.847426 79.233425)
 		(width 0.2)
 		(layer "B.Cu")
@@
 	)
 	(segment
-		(start 89.064428 78.021375)
-		(end 90.132434 78.021375)
+		(start 70.215087 81.2292)
+		(end 69.6848 80.698913)
 		(width 0.2)
 		(layer "B.Cu")
@@
 	)
 	(segment
-		(start 90.132434 78.021375)
-		(end 90.847426 78.736367)
+		(start 72.672842 80.581271)
+		(end 72.024913 81.2292)
 		(width 0.2)
 		(layer "B.Cu")
@@
 	)
 	(segment
-		(start 88.594299 80.6576)
-		(end 80.485586 80.6576)
+		(start 69.87423 95.7708)
+		(end 72.518172 95.7708)
 		(width 0.2)
 		(layer "B.Cu")
@@
 	)
 	(segment
-		(start 78.150685 98.145)
-		(end 78.385 98.379315)
+		(start 88.594299 80.6576)
+		(end 80.485586 80.6576)
 		(width 0.2)
 		(layer "B.Cu")
@@
 	)
 	(segment
-		(start 79.357886 99.695)
-		(end 79.375 99.695)
+		(start 73.803728 96.802357)
+		(end 74.3584 97.35703)
 		(width 0.2)
 		(layer "B.Cu")
@@
 	)
 	(segment
-		(start 75.285 98.895)
-		(end 75.285 98.379315)
+		(start 74.3584 97.35703)
+		(end 74.3584 99.00823)
 		(width 0.2)
 		(layer "B.Cu")
@@
 	)
 	(segment
-		(start 89.538 79.713901)
-		(end 88.594299 80.6576)
+		(start 78.150685 98.145)
+		(end 78.385 98.379315)
 		(width 0.2)
 		(layer "B.Cu")
@@
 	)
 	(segment
-		(start 69.87423 95.7708)
-		(end 72.518172 95.7708)
+		(start 78.385 100.222114)
+		(end 78.607886 100.445)
 		(width 0.2)
 		(layer "B.Cu")
@@
 	)
 	(segment
-		(start 69.6848 80.698913)
-		(end 69.6848 95.96023)
+		(start 75.285 98.379315)
+		(end 75.519315 98.145)
 		(width 0.2)
 		(layer "B.Cu")
@@
 	)
 	(segment
-		(start 78.385 98.379315)
-		(end 78.385 100.222114)
+		(start 80.485586 80.6576)
+		(end 79.587184 81.556)
 		(width 0.2)
 		(layer "B.Cu")
@@
 	)
 	(segment
-		(start 73.549729 96.802357)
-		(end 73.803728 96.802357)
+		(start 74.3584 99.00823)
+		(end 74.47163 98.895)
 		(width 0.2)
 		(layer "B.Cu")
@@
 	)
 	(segment
-		(start 89.538 79.3432)
-		(end 89.538 79.713901)
+		(start 90.132434 78.021375)
+		(end 90.847426 78.736367)
 		(width 0.2)
 		(layer "B.Cu")
@@
 	)
 	(segment
-		(start 69.6848 95.96023)
-		(end 69.87423 95.7708)
+		(start 89.538 79.3432)
+		(end 89.538 79.713901)
 		(width 0.2)
 		(layer "B.Cu")
@@
 	)
 	(segment
-		(start 78.607886 100.445)
-		(end 79.357886 99.695)
+		(start 69.6848 80.698913)
+		(end 69.6848 95.96023)
 		(width 0.2)
 		(layer "B.Cu")
@@
 	)
 	(segment
-		(start 90.847426 78.736367)
-		(end 90.847426 79.233425)
+		(start 73.447571 81.355999)
+		(end 72.672842 80.581271)
 		(width 0.2)
 		(layer "B.Cu")
@@
 	)
 	(segment
-		(start 75.285 98.379315)
-		(end 75.519315 98.145)
+		(start 69.6848 95.96023)
+		(end 69.87423 95.7708)
 		(width 0.2)
 		(layer "B.Cu")
@@
 	)
 	(segment
-		(start 90.495955 79.584896)
-		(end 89.852896 79.584896)
+		(start 73.914 81.355999)
+		(end 73.447571 81.355999)
 		(width 0.2)
 		(layer "B.Cu")
@@
 	)
 	(segment
-		(start 74.114001 81.556)
-		(end 73.914 81.355999)
+		(start 74.47163 98.895)
+		(end 75.285 98.895)
 		(width 0.2)
 		(layer "B.Cu")
@@
 	)
 	(segment
-		(start 89.852896 79.584896)
-		(end 89.6112 79.3432)
+		(start 89.064428 78.021375)
+		(end 90.132434 78.021375)
 		(width 0.2)
 		(layer "B.Cu")
@@
 	)
 	(segment
-		(start 75.519315 98.145)
-		(end 78.150685 98.145)
+		(start 90.847426 79.233425)
+		(end 90.495955 79.584896)
 		(width 0.2)
 		(layer "B.Cu")
